File: Hardware/myPlant.sch (EAGLE design)
At the start: 42 parts, among them IC2 LMV358, Q2 MMBT2222A, SW1 KMR2, SW2 KMR2, U1 FSA3357, U2 NCP1402, U3 ALS-PT19, U6 SI7021, X1 ESP-12

Commit message: Added load switch
Parts:
- removed C10, C18, C19: 0.1uF, SparkFun-Capacitors:0.1UF-25V(+80/-20%)(0603)
- removed D4: WS2812, SparkFun-LED:WS2812B
- removed FID1, FID2: FIDUCIAL1X2, SparkFun-Aesthetics:FIDUCIAL1X2
- removed LOGO2: OSHW-LOGOS, SparkFun-Aesthetics:OSHW-LOGOS
- removed Q2: MMBT2222A, SparkFun-DiscreteSemi:TRANSISTOR_NPNMMBT2222A
- removed R15, R16: 4.7K, SparkFun-Resistors:4.7KOHM-1/10W-1%(0603)
- removed R17: 10K, SparkFun-Resistors:10KOHM1/10W1%(0603)0603
- removed STANDOFF1, STANDOFF2, STANDOFF3, STANDOFF4: STAND-OFF, SparkFun-Electromechanical:STAND-OFF
- removed SW1, SW2: KMR2, microbuilder:SWITCH_TACT_SMT4.6X2.8
- removed U6: SI7021, SparkFun-Sensors:SI7021
- added C3, C6: 0.1uF, SparkFun-Capacitors:0.1UF-0603-25V-(+80/-20%)
- added C5: 10uF, SparkFun:CAP_POL1206
- added C7: 68uF, SparkFun:CAP_POL3528
- added C8: 1.0uF, SparkFun-Capacitors:1.0UF-0603-16V-10%
- added D3: MBRA140, SparkFun:DIODESMA
- added H1, H2, H3, H4: STAND-OFF, SparkFun-Hardware:STAND-OFF
- added IC1: LMV358, SparkFun-AnalogIC:OPAMP-DUALU
- added LOGO1: OSHW-LOGOM, SparkFun-Aesthetics:OSHW-LOGOM
- added R8, R9: 10k, SparkFun-Resistors:10KOHM-0603-1/10W-1%
- added S1: BTN-0, SparkFun-Electromechanical:SWITCH-MOMENTARY-2SMD-4.6X2.8MM
- added S2: RESET, SparkFun-Electromechanical:SWITCH-MOMENTARY-2SMD-4.6X2.8MM
- added SJ1: SLEEP, SparkFun-Passives:JUMPER-PAD-2-NC_BY_TRACE
- added U4: TPS22860, alex:TPS22860
- C1: value 10uF -> 0.1uF; device SparkFun:CAP_POL1206 -> SparkFun-Capacitors:0.1UF-0603-25V-(+80/-20%)
- C2: value 68uF -> 1.0uF; device SparkFun:CAP_POL3528 -> SparkFun-Capacitors:1.0UF-0603-16V-10%
- C4: value 1uF -> 0.1uF; device SparkFun:CAP0603-CAP -> SparkFun-Capacitors:0.1UF-0603-25V-(+80/-20%)
- D1: value MBRA140 -> WS2812; device SparkFun:DIODESMA -> SparkFun-LED:WS2812B
- FRAME1: value FRAME-LEDGER -> FRAME-LETTER; device SparkFun-Aesthetics:FRAME-LEDGER -> SparkFun-Aesthetics:FRAME-LETTER
- IC2: value LMV358 -> NCP1402; device SparkFun-AnalogIC:OPAMP-DUALU -> SparkFun:V_REG_NCP1400SOT23-5; PROD_ID IC-09657 -> (none)
- L1: value 47uH -> 47µH; device SparkFun:INDUCTORCR54 -> SparkFun-Coils:INDUCTOR-CR54-47UH
- R1: value 10K -> 510k; device SparkFun:RESISTOR0603-RES -> SparkFun-Resistors:10KOHM-0603-1/10W-1%
- R10, R12, R5, R6, R7: value 10K -> 10k; device SparkFun-Resistors:10KOHM-1/10W-1%(0603)0603 -> SparkFun-Resistors:10KOHM-0603-1/10W-1%
- R11: value 22K -> 22k; device SparkFun-Resistors:22KOHM1/10W1%(0603) -> SparkFun-Resistors:22KOHM-0603-1/10W-1%
- R2: value 510K -> 10k; device SparkFun:RESISTOR0603-RES -> SparkFun-Resistors:10KOHM-0603-1/10W-1%
- R3, R4: value 10K -> 4.7k; device SparkFun-Resistors:10KOHM-1/10W-1%(0603)0603 -> SparkFun-Resistors:4.7KOHM-0603-1/10W-1%
- U1: value FSA3357 -> SI7021; device alex:FSA3357 -> SparkFun-Sensors:SI7021
- U2: value NCP1402 -> ALS-PT19; device SparkFun:V_REG_NCP1400SOT23-5 -> SparkFun-Sensors:LIGHTSENSORALS
- U3: value ALS-PT19 -> FSA3357; device SparkFun-Sensors:LIGHTSENSORALS -> alex:FSA3357
Connections:
- removed net CAPACITANCE_V: C4.1, D2.C, R2.1, U1.B0
- removed net GPIO0: R5.1, SW2.S, SW2.S1, X1.GPIO0
- removed net GPIO12: R17.1, X1.GPIO12
- removed net GPIO13: U1.S1, X1.GPIO13
- removed net GPIO14: U1.S2, X1.GPIO14
- removed net GPIO15: R1.2, R6.2, X1.GPIO15
- removed net GPIO2: D4.DIN, R7.1, X1.GPIO2
- removed net N$6: Q2.B, R17.2
- new net 0/BUTTON: R5.1, S1.2, X1.GPIO0
- new net 12/S1: U3.S1, X1.GPIO12
- new net 13/S2: U3.S2, X1.GPIO13
- new net 14/PWR: U4.ON, X1.GPIO14
- new net 15/CLK: R10.2, R2.2, X1.GPIO15
- new net 2/WS2812: D1.DIN, R8.1, X1.GPIO2
- new net CAPACITANCE: C2.1, D2.C, R1.2, U3.B0
- new net GPIO16: SJ1.1, X1.GPIO16
- net 3.3V: now also C7.+, C8.1, D3.C, IC2.EN, IC2.OUT, R6.2, R8.2, R9.2, U4.VBIAS, U4.VIN; no longer C2.+, D1.C, Q2.C, R3.2, R4.2, R7.2, U2.EN, U2.OUT
- net 4/SDA: now also R3.1, U1.DATA; no longer R15.1, U6.DATA
- net 5/SCL: now also R4.1, U1.SCK; no longer R16.1, U6.SCK
- net ADC: now also IC1B.-IN, IC1B.OUT; no longer IC2B.-IN, IC2B.OUT
- net ADC-IN: now also IC1A.+IN, U3.A; no longer IC2A.+IN, U1.A
- net CH_PD: now also R9.1; no longer R3.1
- net GND: now also C1.2, C2.2, C3.2, C5.-, C6.2, C7.-, C8.2, D1.VSS, IC1A.V-, IC2.GND, R1.1, R7.1, S1.1, S2.1, U3.GND, U4.GND; no longer C1.-, C10.2, C18.2, C19.2, C2.-, D4.VSS, IC2A.V-, R2.2, R6.1, SW1.P, SW1.P1, SW2.P, SW2.P1, U2.GND, U6.GND
- net LIGHT: now also R7.2, U2.E1, U3.B1; no longer R10.2, U1.B1, U3.E1
- net N$1: now also D3.A, IC2.LX; no longer D1.A, U2.LX
- net N$15: now also IC1A.-IN, IC1A.OUT; no longer IC2A.-IN, IC2A.OUT
- net N$18: now also IC1B.+IN; no longer IC2B.+IN
- net RAW: now also C5.+, U3.B2; no longer C1.+, U1.B2
- net RESET: now also R6.1, S2.2, SJ1.2; no longer R4.1, SW1.S, SW1.S1, X1.GPIO16
- net VCC: now also C1.1, C3.1, C4.1, C6.1, D1.VDD, IC1A.V+, R3.2, R4.2, U1.VDD, U2.C1, U3.VCC, U4.VOUT; no longer C10.1, C18.1, C19.1, D4.VDD, IC2A.V+, Q2.E, R15.2, R16.2, U1.VCC, U3.C1, U6.VDD
- net V_CAP: now also R2.1; no longer R1.1
Other:
- note added: "Capacitive Soil Moisture Sensor"
- note added: "FTDI Connector"
- note added: "GPIO0 Button"
- note added: "Load Switch"
- note added: "Reset Button"
- note added: "Run Default Pull-Ups"
- note added: "SJ2 can be cut to disable the sleep mode feature"
- note added: "Sleep Mode"
- note added: "WiFi Module"
- note removed: "Battery Level"
- note removed: "Capacitive soil moisture sensor"
- note removed: "ESP8266"
- moved on the sheet: BAT1, C4, D2, JP1, R1, R10, R11, R12, R2, R3, R4, R5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

Commit message: Done preliminary pcb placement
Parts:
- removed C5: 10uF, SparkFun:CAP_POL1206
- removed C7: 68uF, SparkFun:CAP_POL3528
- removed D3: MBRA140, SparkFun:DIODESMA
- removed H1, H2, H3, H4: STAND-OFF, SparkFun-Hardware:STAND-OFF
- removed IC1: LMV358, SparkFun-AnalogIC:OPAMP-DUALU
- removed IC2: NCP1402, SparkFun:V_REG_NCP1400SOT23-5
- removed L1: 47µH, SparkFun-Coils:INDUCTOR-CR54-47UH
- added C10: 68uF, SparkFun:CAP_POL3528
- added C9: 10uF, SparkFun:CAP_POL1206
- added D4: MBRA140, SparkFun:DIODESMA
- added L2: 47uH, SparkFun:INDUCTORCR54
- added U5: NCP1402, SparkFun:V_REG_NCP1400SOT23-5
- added U6: (no value), SparkFun-IC-Amplifiers:LMV358
Connections:
- removed net N$1: D3.A, IC2.LX, L1.2
- removed net RAW: BAT1.+, C5.+, L1.1, U3.B2
- new net N$3: D4.A, L2.2, U5.LX
- new net VBAT: BAT1.+, C9.+, L2.1, U3.B2
- net 3.3V: now also C10.+, D4.C, U5.EN, U5.OUT; no longer C7.+, D3.C, IC2.EN, IC2.OUT
- net ADC: now also U6G2.-IN, U6G2.OUT; no longer IC1B.-IN, IC1B.OUT
- net ADC-IN: now also U6G1.+IN; no longer IC1A.+IN
- net GND: now also C10.-, C9.-, U5.GND, U6G3.P$V-; no longer C5.-, C7.-, IC1A.V-, IC2.GND
- net N$15: now also U6G1.-IN, U6G1.OUT; no longer IC1A.-IN, IC1A.OUT
- net N$18: now also U6G2.+IN; no longer IC1B.+IN
- net VCC: now also U6G3.P$V+; no longer IC1A.V+
